Commit message: fix: hand-eye 캘리브레이션 버그 수정 및 planning_node 안정성 개선
- nero_with_camera.urdf: d435_camera_joint가 실제 tf2 체인의 수정 대상임을
  확인, y 오프셋 보정(-0.028 → 0.012) 적용 (임시값, 재캘리브레이션 필요)
- calib_visual.py: 새 hand-eye 캘리브레이션 스크립트 추가 (RViz 시각화 포함)
  주의: _apply_to_urdf()가 주석 내 joint를 패치하는 버그 있음 → 수동 보정 필요
- launch/rsp.launch.py: robot_state_publisher 런치파일 추가
- planning_node.py: 급회전 안전정지 임시 비활성화(속도 0.15로 완화),
  from_scan 시 align 각도 재조회 활성화, _abs_angle_to_quat 함수 추가
- docs/wiki: 캘리브레이션 이력/d435_camera_joint 수정 위치/재캘리브 가이드 추가

Co-Authored-By: Claude Sonnet 4.6 <noreply@anthropic.com>

File: sj_pickplace/nero_with_camera.urdf (robot description, URDF)
Before this commit: robot agx_arm, 19 links, 18 joints
Joints:
- joint d435_camera_joint: origin xyz=-0.031 -0.028 0.0018 rpy=0.0 -1.22 0.0 -> xyz=-0.031 0.012 0.0018 rpy=0.0 -1.22 0.0
